File: GardenGuard/GardenGuard.sch (KiCad schematic (older format))
At the start: 9 parts

Commit message: Added powersupply stages
Parts:
- removed BT?: Battery_Cell, symbol Device:Battery_Cell
- removed D?: D_Schottky_Small, symbol Device:D_Schottky_Small
- removed D?: D_Small, symbol Device:D_Small
- removed U?: ESP32-WROOM-32, RF_Module:ESP32-WROOM-32, symbol RF_Module:ESP32-WROOM-32
- added BT1, BT2: LiOn, Battery:BatteryHolder_Keystone_1042_1x18650, symbol Device:Battery_Cell
- added BZ1: Buzzer, Buzzer_Beeper:Buzzer_12x9.5RM7.6, symbol Device:Buzzer
- added C1, C2, C3: 10nF, Capacitor_SMD:C_0805_2012Metric_Pad1.18x1.45mm_HandSolder, symbol Device:C_Small
- added C14, C15, C5: 0.1uF, Capacitor_SMD:C_0805_2012Metric_Pad1.18x1.45mm_HandSolder, symbol Device:C_Small
- added C16, C17, C18, C4: 10uF, Capacitor_SMD:C_0805_2012Metric_Pad1.18x1.45mm_HandSolder, symbol Device:C_Small
- added D1, D2, D8: R, LED_SMD:LED_0805_2012Metric_Castellated, symbol Device:LED_Small
- added D7: 1N5819, Diode_SMD:D_SOD-123, symbol Device:D_Schottky_Small
- added D9: B, LED_SMD:LED_0805_2012Metric_Castellated, symbol Device:LED_Small
- added J2: OLED SSD1306, Connector_PinHeader_2.54mm:PinHeader_1x04_P2.54mm_Vertical, symbol Connector_Generic:Conn_01x04
- added Q3: FQP27P06, Package_TO_SOT_SMD:SOT-23, symbol Device:Q_PMOS_DGS
- added R1: 220k, Resistor_SMD:R_0805_2012Metric_Pad1.20x1.40mm_HandSolder, symbol Device:R_Small
- added R10, R9: 330R, Resistor_SMD:R_0805_2012Metric_Pad1.20x1.40mm_HandSolder, symbol Device:R_Small
- added R2, R25, R3, R4, R5, R6, R7: 100k, Resistor_SMD:R_0805_2012Metric_Pad1.20x1.40mm_HandSolder, symbol Device:R_Small
- added R24: 4.7K, Resistor_SMD:R_0805_2012Metric_Pad1.20x1.40mm_HandSolder, symbol Device:R_Small
- added R26, R27, R29, R30, R?: 1K, Resistor_SMD:R_0805_2012Metric_Pad1.20x1.40mm_HandSolder, symbol Device:R_Small
- added R28: 100, Resistor_SMD:R_0805_2012Metric_Pad1.20x1.40mm_HandSolder, symbol Device:R_Small
- added R8: NC, Resistor_SMD:R_0805_2012Metric_Pad1.20x1.40mm_HandSolder, symbol Device:R_Small
- added RV1: 10K, Potentiometer_SMD:Potentiometer_Bourns_3224J_Horizontal, symbol Device:R_POT_Small
- added SW1: Reset, Button_Switch_SMD:SW_SPST_B3U-3000P, symbol Switch:SW_Push
- added SW2: SW_Push, Button_Switch_SMD:SW_SPST_B3U-3000P, symbol Switch:SW_Push
- added U1: ESP-07, RF_Module:ESP-07, symbol RF_Module:ESP-07
- added U2: DS18B20, Package_TO_SOT_THT:TO-92_Inline, symbol Sensor_Temperature:DS18B20
- added U4: TP4056, Project_footprints:TP4056_SOP-8-PP, symbol custom:TP4056
- added U5: FS8205A, Package_SO:TSSOP-8_4.4x3mm_P0.65mm, symbol custom:FS8205A
- added U6: DW01A, Package_TO_SOT_SMD:SOT-23-6, symbol custom:DW01A
- added U7: HT75xx-1-SOT89, Package_TO_SOT_SMD:SOT-89-3, symbol Regulator_Linear:HT75xx-1-SOT89
- C6: renamed from C?; value C_Small -> 0.1uF; footprint (none) -> Capacitor_SMD:C_0805_2012Metric_Pad1.18x1.45mm_HandSolder
- J1: renamed from J?; value Conn_01x02 -> Sollar; footprint (none) -> Connector_JST:JST_VH_B2P-VH-B_1x02_P3.96mm_Vertical
- J3: renamed from J?; footprint (none) -> Connector_Audio:Jack_3.5mm_Ledino_KB3SPRS_Horizontal
- R11: renamed from R?; footprint (none) -> Resistor_SMD:R_0805_2012Metric_Pad1.20x1.40mm_HandSolder
- SW3: renamed from SW?; footprint (none) -> Rotary_Encoder:RotaryEncoder_Alps_EC11E-Switch_Vertical_H20mm
Connections:
- net labels added: +3.3V, ACD, ADC1, EN, GND, GND1, GPIO0, GPIO12, GPIO13, GPIO14, GPIO15, GPIO2, RXD, Reset, SCL, SDA, TXD, VCC, WAKE
- wire segments 0 -> 160
- no-connect marks 0 -> 3
Other:
- moved on the sheet: C6, J1, J3, R11, SW3

Commit message: shematic finished
Parts:
- added C10, C8, C9, C?: 10nF, Capacitor_SMD:C_0805_2012Metric_Pad1.18x1.45mm_HandSolder, symbol Device:C_Small
- added C7: 10n, Capacitor_SMD:C_0805_2012Metric_Pad1.18x1.45mm_HandSolder, symbol Device:C_Small
- added D3, D4: D_TVS, Diode_SMD:D_0805_2012Metric_Castellated, symbol Device:D_TVS
- added J4: USB_B_Mini, Connector_USB:USB_Micro-B_Amphenol_10118194_Horizontal, symbol Connector:USB_B_Mini
- added Q1: RE1C002UN, symbol Device:Q_NMOS_GSD
- added Q2: BC548, Package_TO_SOT_THT:TO-92_Inline, symbol Transistor_BJT:BC548
- added R12: 0R, Resistor_SMD:R_0805_2012Metric_Pad1.20x1.40mm_HandSolder, symbol Device:R_Small
- added R13: 100K, Resistor_SMD:R_0805_2012Metric_Pad1.20x1.40mm_HandSolder, symbol Device:R_Small
- added R14, R15, R16, R17, R?: 10K, Resistor_SMD:R_0805_2012Metric_Pad1.20x1.40mm_HandSolder, symbol Device:R_Small
- R1: value 220k -> 220K
- R11: value R_Small -> 1M
- R2, R4, R5, R7: value 100k -> 100K
- R28: value 100 -> 100R
- R3: value 100k -> 1K
- gave numbers to parts that had none: 1
Connections:
- net labels added: BOOT, BUZZ, B_CHECK, LED, ROT_A, ROT_B, ROT_S, SHIELD, VBUS, V_BAT
- net labels removed: ACD
- wire segments 160 -> 225
Other:
- moved on the sheet: BT1, BT2, BZ1, C1, C14, C15, C16, C17, C18, C2, C3, C4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

Commit message: Updated packages, start layout
Parts:
- removed C?: 10nF, Capacitor_SMD:C_0805_2012Metric_Pad1.18x1.45mm_HandSolder, symbol Device:C_Small
- removed D3, D4: D_TVS, Diode_SMD:D_0805_2012Metric_Castellated, symbol Device:D_TVS
- removed J3: AudioJack4_Ground_SwitchTR1, Connector_Audio:Jack_3.5mm_Ledino_KB3SPRS_Horizontal, symbol Connector:AudioJack4_Ground_SwitchTR1
- removed R?: 10K, Resistor_SMD:R_0805_2012Metric_Pad1.20x1.40mm_HandSolder, symbol Device:R_Small
- removed SW2: SW_Push, Button_Switch_SMD:SW_SPST_B3U-3000P, symbol Switch:SW_Push
- added C14: 0.1uF, Capacitor_SMD:C_0805_2012Metric_Pad1.18x1.45mm_HandSolder, symbol Device:C_Small
- added H1, H2, H3, H4: MountingHole, MountingHole:MountingHole_3.2mm_M3_DIN965, symbol Mechanical:MountingHole
- added J3: PJ-321A, Project_footprints:PJ-321A, symbol pj:PJ-321A
- added J5: DEBUG, Connector_PinHeader_2.54mm:PinHeader_1x04_P2.54mm_Vertical, symbol Connector_Generic:Conn_01x04
- added JP1: BOOT, Jumper:SolderJumper-2_P1.3mm_Open_RoundedPad1.0x1.5mm, symbol Device:Jumper_NO_Small
- C3: renamed from C16; footprint Capacitor_SMD:C_0805_2012Metric_Pad1.18x1.45mm_HandSolder -> Capacitor_SMD:C_1206_3216Metric_Pad1.33x1.80mm_HandSolder
- J1: footprint Connector_JST:JST_VH_B2P-VH-B_1x02_P3.96mm_Vertical -> Project_footprints:ER-CON2.0-2P-SMD
- Q1: footprint (none) -> Package_TO_SOT_SMD:SOT-23_Handsoldering
- Q3: renamed from Q2; footprint Package_TO_SOT_THT:TO-92_Inline -> Package_TO_SOT_SMD:SOT-23
- renumbered BT2 to BT1, BT1 to BT2, C7 to C1, C4 to C10, C5 to C11, C18 to C12, C8 to C13, C9 to C15, C10 to C16, C14 to C2, C6 to C4, C1 to C5, C15 to C6, C2 to C7, C3 to C8, C17 to C9, D8 to D2, D9 to D3, D7 to D5, D1 to D6, D2 to D7, J4 to J2, J2 to J4, Q3 to Q2, R11 to R1, R1 to R10, R2 to R11, R3 to R12, R28 to R13, R4 to R14, R5 to R15, R25 to R16, R6 to R17, R7 to R18, R8 to R19, R12 to R2, R14 to R21, R15 to R22, R16 to R23, R17 to R24, R9 to R25, R10 to R26, R29 to R3, R30 to R4, R26 to R5, R31 to R6, R13 to R7, R24 to R8, R27 to R9, U4 to U1, U6 to U3, U5 to U4, U1 to U5, U7 to U6
Connections:
- net VBUS is gone; now on net VCC: R2.1
- net +3V3: now also C14.2, J3.2, J5.1 (Pin_1)
- net GND: now also C14.1, J3.1, J5.4 (Pin_4), JP1.2
- net GPIO0: now also JP1.1
- net GPIO13: now also J3.3
- net RXD: now also J5.2 (Pin_2)
- net TXD: now also J5.3 (Pin_3)
- no-connect marks 3 -> 6
Other:
- moved on the sheet: C13, C15, C16, J4, R21, R22, R23, SW3

Commit message: layout done
Parts:
- removed Q2: FQP27P06, Package_TO_SOT_SMD:SOT-23, symbol Device:Q_PMOS_DGS
- removed Q3: BC548, Package_TO_SOT_SMD:SOT-23, symbol Transistor_BJT:BC548
- added C17: 0.1uF, Capacitor_SMD:C_1206_3216Metric_Pad1.33x1.80mm_HandSolder, symbol Device:C_Small
- added Q2: FQP27P06, Package_TO_SOT_SMD:SOT-23_Handsoldering, symbol Device:Q_PMOS_GSD
- added Q3: Q_NPN_BEC, Package_TO_SOT_SMD:SOT-23_Handsoldering, symbol Device:Q_NPN_BEC
- C10, C2: footprint Capacitor_SMD:C_0805_2012Metric_Pad1.18x1.45mm_HandSolder -> Capacitor_SMD:C_1206_3216Metric_Pad1.33x1.80mm_HandSolder
Connections:
- net B_CHECK: now also U5.5 (GPIO14); no longer U5.6 (GPIO12)
- net GND: now also J1.1 (Pin_1), C17.1, Q3.2 (E); no longer J1.2 (Pin_2)
- net GPIO13: no longer J3.3, R8.2, U2.2 (DQ)
- net VCC: now also J1.2 (Pin_2), C17.2, Q2.1 (G); no longer J1.1 (Pin_1)
- net V_BAT: now also Q2.3 (D)
- net at BZ1.2 (+): now also Q3.3 (C)
- net at C9.1, D5.1 (K), U6.2 (VIN): now also Q2.2 (S)
- net dw01a_od: now reaches U3.1 (OD), U4.4 (G1)
- net dw01a_cs: now reaches R9.1, U3.2 (CS)
- net dw01a_oc: now reaches U3.3 (OC), U4.5 (G2)
- net dw01a_vcc: now reaches C6.1, R13.2, U3.5 (VCC)
- net T_BAT: now reaches U1.1 (TEMP)
- net prog: now reaches R5.1, U1.2 (PROG)
- net at R24.2: now also Q3.1 (B)
- net GPIO14 renamed GPIO12
- net GPIO12: now also J3.3, R8.2, U2.2 (DQ), U5.6 (GPIO12); no longer U5.5 (GPIO14)
Changed lines of the file:
@@
 Sheet 1 1
 Title "GardenGuard"
-Date "2021-07-22"
+Date "2021-07-24"
 Rev "v0.1.0"
 Comp "Juraj Giertl"
@@
 L Connector_Generic:Conn_01x02 J1
 U 1 1 60982955
-P 950 1200
-F 0 "J1" H 1030 1192 50  0000 L CNN
-F 1 "Sollar" H 1030 1101 50  0000 L CNN
-F 2 "Project_footprints:ER-CON2.0-2P-SMD" H 950 1200 50  0001 C CNN
-F 3 "~" H 950 1200 50  0001 C CNN
-	1    950  1200
-	-1   0    0    -1
+P 950 1300
+F 0 "J1" H 1030 1292 50  0000 L CNN
+F 1 "Sollar" H 1030 1201 50  0000 L CNN
+F 2 "Project_footprints:ER-CON2.0-2P-SMD" H 950 1300 50  0001 C CNN
+F 3 "~" H 950 1300 50  0001 C CNN
+	1    950  1300
+	-1   0    0    1
 $EndComp
 $Comp
@@
 Wire Wire Line
 	6350 4550 6950 4550
-Wire Wire Line
-	6350 4650 6950 4650
 Wire Wire Line
 	6350 4750 6950 4750
@@
 F 0 "C10" V 6000 3650 50  0000 L CNN
 F 1 "10uF" V 6000 3350 50  0000 L CNN
-F 2 "Capacitor_SMD:C_0805_2012Metric_Pad1.18x1.45mm_HandSolder" H 5950 3600 50  0001 C CNN
+F 2 "Capacitor_SMD:C_1206_3216Metric_Pad1.33x1.80mm_HandSolder" H 5950 3600 50  0001 C CNN
 F 3 "~" H 5950 3600 50  0001 C CNN
 	1    5950 3600
@@
 $EndComp
 Text Label 2750 7000 2    50   ~ 0
-GPIO13
+ONE_WIRE
 $Comp
 L Device:Battery_Cell BT2
@@
 	1    5200 2050
 	1    0    0    -1
-$EndComp
-$Comp
-L Device:Q_PMOS_DGS Q2
-U 1 1 61063B11
-P 5450 1100
-F 0 "Q2" V 5400 950 50  0000 C CNN
-F 1 "FQP27P06" V 5700 1100 50  0000 C CNN
-F 2 "Package_TO_SOT_SMD:SOT-23" H 5650 1200 50  0001 C CNN
-F 3 "~" H 5450 1100 50  0001 C CNN
-	1    5450 1100
-	0    -1   1    0
 $EndComp
 $Comp
@@
 F 0 "C2" H 1592 1496 50  0000 L CNN
 F 1 "0.1uF" H 1592 1405 50  0000 L CNN
-F 2 "Capacitor_SMD:C_0805_2012Metric_Pad1.18x1.45mm_HandSolder" H 1500 1450 50  0001 C CNN
+F 2 "Capacitor_SMD:C_1206_3216Metric_Pad1.33x1.80mm_HandSolder" H 1500 1450 50  0001 C CNN
 F 3 "~" H 1500 1450 50  0001 C CNN
 	1    1500 1450
@@
 	10250 1550 10250 1600
 $Comp
-L Transistor_BJT:BC548 Q3
-U 1 1 619D6D28
-P 10150 1800
-F 0 "Q3" H 10341 1846 50  0000 L CNN
-F 1 "BC548" H 10341 1755 50  0000 L CNN
-F 2 "Package_TO_SOT_SMD:SOT-23" H 10350 1725 50  0001 L CIN
-F 3 "https://www.onsemi.com/pub/Collateral/BC550-D.pdf" H 10150 1800 50  0001 L CNN
-	1    10150 1800
-	1    0    0    -1
-$EndComp
-$Comp
 L Device:R_Small R24
 U 1 1 619D9812
@@
 Wire Wire Line
 	6800 3750 6800 3500
-Text GLabel 6950 4650 2    50   Output ~ 0
-B_CHECK
 Text Label 4850 1200 0    50   ~ 0
 V_BAT
@@
 Text Label 6950 4050 0    50   ~ 0
 ROT_S
-Text Label 6950 4850 0    50   ~ 0
+Text Label 7400 4650 0    50   ~ 0
 ROT_B
 Text Label 6950 4750 0    50   ~ 0
@@
 	1650 6850 1800 6850
 Text Label 1900 6750 0    50   ~ 0
-GPIO13
+ONE_WIRE
 Wire Wire Line
 	1650 6750 1900 6750
@@
 NoConn ~ 1250 3900
 NoConn ~ 1250 4000
+$Comp
+L Device:Q_NPN_BEC Q3
+U 1 1 6101ABC4
+P 10150 1800
+F 0 "Q3" H 10341 1846 50  0000 L CNN
+F 1 "Q_NPN_BEC" H 10341 1755 50  0000 L CNN
+F 2 "Package_TO_SOT_SMD:SOT-23_Handsoldering" H 10350 1900 50  0001 C CNN
+F 3 "~" H 10150 1800 50  0001 C CNN
+	1    10150 1800
+	1    0    0    -1
+$EndComp
+$Comp
+L Device:Q_PMOS_GSD Q2
+U 1 1 610925FE
+P 5450 1100
+F 0 "Q2" V 5699 1100 50  0000 C CNN
+F 1 "FQP27P06" V 5790 1100 50  0000 C CNN
+F 2 "Package_TO_SOT_SMD:SOT-23_Handsoldering" H 5650 1200 50  0001 C CNN
+F 3 "~" H 5450 1100 50  0001 C CNN
+	1    5450 1100
+	0    -1   1    0
+$EndComp
+Text Label 6950 4650 0    50   ~ 0
+ONE_WIRE
+Text Label 6950 4850 0    50   ~ 0
+B_CHECK
+Wire Wire Line
+	6350 4650 7400 4650
+Text Label 3350 1750 0    11   ~ 0
+dw01a_cs
+Text Label 2900 1850 0    11   ~ 0
+prog
+Text Label 2950 1750 0    50   ~ 0
+T_BAT
+Wire Wire Line
+	2900 1750 2950 1750
+Text Label 3750 2000 0    11   ~ 0
+dw01a_oc
+Text Label 3950 2000 0    11   ~ 0
+dw01a_od
+Text Label 4350 1500 0    11   ~ 0
+dw01a_vcc
+$Comp
+L Device:C_Small C17
+U 1 1 61280119
+P 4150 850
+F 0 "C17" H 4242 896 50  0000 L CNN
+F 1 "0.1uF" H 4242 805 50  0000 L CNN
+F 2 "Capacitor_SMD:C_1206_3216Metric_Pad1.33x1.80mm_HandSolder" H 4150 850 50  0001 C CNN
+F 3 "~" H 4150 850 50  0001 C CNN
+	1    4150 850
+	0    -1   1    0
+$EndComp
+$Comp
+L power:VCC #PWR0107
+U 1 1 61280369
+P 4250 850
+F 0 "#PWR0107" H 4250 700 50  0001 C CNN
+F 1 "VCC" H 4265 1023 50  0000 C CNN
+F 2 "" H 4250 850 50  0001 C CNN
+F 3 "" H 4250 850 50  0001 C CNN
+	1    4250 850
+	0    1    1    0
+$EndComp
+$Comp
+L power:GND #PWR0108
+U 1 1 612809B5
+P 4050 850
+F 0 "#PWR0108" H 4050 600 50  0001 C CNN
+F 1 "GND" H 4055 677 50  0000 C CNN
+F 2 "" H 4050 850 50  0001 C CNN
+F 3 "" H 4050 850 50  0001 C CNN
+	1    4050 850
+	0    1    1    0
+$EndComp
 $EndSCHEMATC

Commit message: Release v1.0.0 - board finished
Parts:
- added R20: 0R, Resistor_SMD:R_0805_2012Metric_Pad1.20x1.40mm_HandSolder, symbol Device:R_Small
- added R27, R28: 1K, Resistor_SMD:R_0805_2012Metric_Pad1.20x1.40mm_HandSolder, symbol Device:R_Small
- added TH1: Thermistor_NTC, Resistor_THT:R_Axial_DIN0204_L3.6mm_D1.6mm_P5.08mm_Horizontal, symbol Device:Thermistor_NTC
Connections:
- net GND: now also R28.2, TH1.2
- net T_BAT: now also R27.2, R28.1, TH1.1
- net VCC: now also R20.1, R27.1; no longer J1.2 (Pin_2)
- new net: J1.2 (Pin_2), R20.2
Changed lines of the file:
@@
 Sheet 1 1
 Title "GardenGuard"
-Date "2021-07-24"
-Rev "v0.1.0"
+Date "2021-07-25"
+Rev "v1.0.0"
 Comp "Juraj Giertl"
 Comment1 "j74a8g@gmail.com"
@@
 $EndComp
 Wire Wire Line
-	1150 1200 1500 1200
+	1150 1200 1200 1200
 $Comp
 L power:GND #PWR03
@@
 	0    1    1    0
 $EndComp
+$Comp
+L Device:R_Small R28
+U 1 1 60FE44B9
+P 5600 2450
+F 0 "R28" H 5659 2496 50  0000 L CNN
+F 1 "1K" H 5659 2405 50  0000 L CNN
+F 2 "Resistor_SMD:R_0805_2012Metric_Pad1.20x1.40mm_HandSolder" H 5600 2450 50  0001 C CNN
+F 3 "~" H 5600 2450 50  0001 C CNN
+	1    5600 2450
+	1    0    0    -1
+$EndComp
+$Comp
+L Device:R_Small R27
+U 1 1 60FE4A53
+P 5600 2000
+F 0 "R27" H 5659 2046 50  0000 L CNN
+F 1 "1K" H 5659 1955 50  0000 L CNN
+F 2 "Resistor_SMD:R_0805_2012Metric_Pad1.20x1.40mm_HandSolder" H 5600 2000 50  0001 C CNN
+F 3 "~" H 5600 2000 50  0001 C CNN
+	1    5600 2000
+	1    0    0    -1
+$EndComp
+$Comp
+L Device:Thermistor_NTC TH1
+U 1 1 60FE56CC
+P 5900 2350
+F 0 "TH1" H 5998 2396 50  0000 L CNN
+F 1 "Thermistor_NTC" H 5998 2305 50  0000 L CNN
+F 2 "Resistor_THT:R_Axial_DIN0204_L3.6mm_D1.6mm_P5.08mm_Horizontal" H 5900 2400 50  0001 C CNN
+F 3 "~" H 5900 2400 50  0001 C CNN
+	1    5900 2350
+	1    0    0    -1
+$EndComp
+$Comp
+L power:GND #PWR0109
+U 1 1 60FE5EC7
+P 5600 2600
+F 0 "#PWR0109" H 5600 2350 50  0001 C CNN
+F 1 "GND" H 5605 2427 50  0000 C CNN
+F 2 "" H 5600 2600 50  0001 C CNN
+F 3 "" H 5600 2600 50  0001 C CNN
+	1    5600 2600
+	1    0    0    -1
+$EndComp
+Wire Wire Line
+	5600 2550 5600 2600
+Wire Wire Line
+	5600 2350 5600 2150
+Wire Wire Line
+	5600 1900 5600 1850
+Wire Wire Line
+	5900 2200 5900 2150
+Wire Wire Line
+	5900 2150 5600 2150
+Connection ~ 5600 2150
+Wire Wire Line
+	5600 2150 5600 2100
+Wire Wire Line
+	5900 2500 5900 2600
+$Comp
+L power:GND #PWR0110
+U 1 1 6108C869
+P 5900 2600
+F 0 "#PWR0110" H 5900 2350 50  0001 C CNN
+F 1 "GND" H 5905 2427 50  0000 C CNN
+F 2 "" H 5900 2600 50  0001 C CNN
+F 3 "" H 5900 2600 50  0001 C CNN
+	1    5900 2600
+	1    0    0    -1
+$EndComp
+Wire Wire Line
+	5900 2150 6100 2150
+Connection ~ 5900 2150
+Text Label 6100 2150 0    50   ~ 0
+T_BAT
+$Comp
+L power:VCC #PWR0111
+U 1 1 6109C615
+P 5600 1850
+F 0 "#PWR0111" H 5600 1700 50  0001 C CNN
+F 1 "VCC" H 5615 2023 50  0000 C CNN
+F 2 "" H 5600 1850 50  0001 C CNN
+F 3 "" H 5600 1850 50  0001 C CNN
+	1    5600 1850
+	1    0    0    -1
+$EndComp
+$Comp
+L Device:R_Small R?
+U 1 1 6109CF5F
+P 1300 1200
+AR Path="/609880F0/6109CF5F" Ref="R?"  Part="1"
+AR Path="/6109CF5F" Ref="R20"  Part="1"
+F 0 "R20" V 1104 1200 50  0000 C CNN
+F 1 "0R" V 1195 1200 50  0000 C CNN
+F 2 "Resistor_SMD:R_0805_2012Metric_Pad1.20x1.40mm_HandSolder" H 1300 1200 50  0001 C CNN
+F 3 "~" H 1300 1200 50  0001 C CNN
+	1    1300 1200
+	0    1    1    0
+$EndComp
+Wire Wire Line
+	1400 1200 1500 1200
 $EndSCHEMATC
